File: pcb/RemoteStation/bus.kicad_sch (KiCad schematic)
At the start: 13 parts, among them J5 Barrel_Jack_Switch, U1 USBLC6-2SC6, U2 FE1.1s, U3 TPS62933, Y1 12MHz

Commit message: update
Connections:
- net +5V: now also U3.6 (BST)
- no-connect marks 7 -> 9

Commit message: update scripts
Parts:
- added C10, C9: 22u, symbol Device:C
- added C11, C8: 100n, symbol Device:C
- added C12: 10u, symbol Device:C
- added L1: L_Iron, symbol Device:L_Iron
- added R2: 49R9, Resistor_SMD:R_0805_2012Metric, symbol Device:R
- added R3: 53k6, Resistor_SMD:R_0805_2012Metric, symbol Device:R
- added R4: 10k2, Resistor_SMD:R_0805_2012Metric, symbol Device:R
Connections:
- net +5V: now also C10.2, C11.2, C9.2, L1.2, R2.1; no longer U3.6 (BST)
- net GND: now also C10.1, C11.1, C12.2, C9.1, R4.2
- net VCC: now also C12.1
- net at U3.5 (SW): now also C8.2, L1.1
- net at U3.8 (FB): now also R3.2, R4.1
- new net: C8.1, U3.6 (BST)
- new net: R2.2, R3.1
- no-connect marks 9 -> 7
Other:
- note added: "5V Power Supply"
- note added: "Power Connector"
- note added: "USB Hub"
- moved on the sheet: C4, C5, C6, C7, J5, U3

Commit message: big update
Parts:
- renumbered C12 to C201, C1 to C202, C4 to C203, C5 to C204, C2 to C205, C6 to C206, C3 to C207, C7 to C208, C8 to C209, C9 to C210, C10 to C211, C11 to C212, J5 to J201, L1 to L201, R1 to R201, R2 to R202, R3 to R203, R4 to R204, U1 to U201, U2 to U202, U3 to U203, Y1 to Y201
Connections:
- net VCC renamed +12V
Other:
- note removed: "5V Power Supply"
- note removed: "Power Connector"
- note removed: "USB Hub"

Commit message: add hash and title
Other:
- note added: "Amateurfunkclub fuer Remote Stationen"
- note added: "Bus"
- note added: "Remote Station"
Changed lines of the file:
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@@
+		)
+	)
+	(text "Remote Station"
+		(exclude_from_sim no)
+		(at 178.816 171.196 0)
+		(effects
+			(font
+				(size 5 5)
+			)
+			(justify left)
+		)
+	)
+	(text "Amateurfunkclub fuer Remote Stationen"
+		(exclude_from_sim no)
+		(at 186.436 189.992 0)
+		(effects
+			(font
+				(size 1.27 1.27)
+			)
+			(justify left)
+		)
+	)
+	(text "Bus"
+		(exclude_from_sim no)
+		(at 179.07 178.054 0)
+		(effects
+			(font
+				(size 4 4)
+			)
+			(justify left)
 		)
 	)

Commit message: add hash
Other:
- note added: "<<HASH>>"
Changed lines of the file:
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@@
+		)
+	)
+	(text "<<HASH>>"
+		(exclude_from_sim no)
+		(at 267.97 193.548 0)
+		(effects
+			(font
+				(size 1.27 1.27)
+			)
+			(justify left)
 		)
 	)
