File: pcb/RemoteStation/raspberry_pi.kicad_sch (KiCad schematic)
At the start: 0 parts

Commit message: big update
Parts:
- added C301, C302, C303: 100n, symbol Device:C
- added D301, D302: LED, symbol Device:LED
- added J301: Conn_01x02, symbol Connector_Generic:Conn_01x02
- added J302, J305: DF40C-100DS-0.4V_51_, DF40C-100DS-0.4V_51_:HIROSE_DF40C-100DS-0.4V_51_, symbol DF40C-100DS-0.4V_51_:DF40C-100DS-0.4V_51_
- added J303: HR911130A, Connector_RJ:RJ45_Pulse_JK0654219NL_Horizontal, symbol HR911130A:HR911130A
- added J304: Micro_SD_Card, symbol Connector:Micro_SD_Card
- added R301, R302: 470, symbol Device:R
- added R303, R305: 1k, symbol Device:R
- added R304: 12k, symbol Device:R
- added R306: 2k2, symbol Device:R
- added U301, U302: TPD4EUSB30, Package_SON:USON-10_2.5x1.0mm_P0.5mm, symbol Power_Protection:TPD4EUSB30
- added U303: SN74LV1T34DBV, Package_TO_SOT_SMD:SOT-23-5, symbol Logic_LevelTranslator:SN74LV1T34DBV
- added U304: RT9742GGJ5, Package_TO_SOT_SMD:TSOT-23-5, symbol Power_Management:RT9742AGJ5F
Connections:
- new net: C301.2, J303.1 (P1)
- new net: J305.1, R306.2
- new net: J301.2 (Pin_2), J302.93
- new net: D302.1 (K), R305.1
- new net: R305.2, U303.4 (Y)
- new net: J303.12, R301.2
- new net: J303.13, R302.1
- new net: D301.1 (K), R303.1
- new net +3V3: C302.1, D301.2 (A), D302.2 (A), J302.78, J302.84, J302.86, J303.11, J303.14, R304.1, U303.5 (VCC), U304.5 (VIN)
- new net +5V: J302.77, J302.79, J302.81, J302.83, J302.85, J302.87
- new net ETH_GREEN: J302.17, R301.1
- new net ETH_YELLOW: J302.15, R302.2
- new net GND: C301.1, C302.2, C303.2, J301.1 (Pin_1), J302.1, J302.13, J302.14, J302.2, J302.22, J302.23, J302.32, J302.33, J302.42, J302.43, J302.52, J302.53, J302.59, J302.60, J302.65, J302.66, J302.7, J302.71, J302.74, J302.8, J302.89, J302.91, J302.98, J303.10 (P10), J303.S1 (SHIELD), J303.S2 (SHIELD), J304.6 (VSS), J304.9 (SHIELD), J305.13, J305.14, J305.19, J305.20, J305.25, J305.26, J305.31, J305.32, J305.37, J305.38, J305.44, J305.50, J305.55, J305.56, J305.61, J305.62, J305.67, J305.68, J305.7, J305.73, J305.74, J305.79, J305.8, J305.80, J305.85, J305.86, J305.91, J305.92, J305.97, J305.98, U301.3 (GND), U301.8 (GND), U302.3 (GND), U302.8 (GND), U303.3 (GND), U304.2 (GND)
- new net LED_nACTIVITY: J302.21, R303.2
- new net LED_nPWR: J302.95, U303.2 (A)
- new net SD_CLK: J302.57, J304.5 (CLK)
- new net SD_CMD: J302.62, J304.3 (CMD)
- new net SD_DATA0: J302.63, J304.7 (DAT0)
- new net SD_DATA1: J302.67, J304.8 (DAT1)
- new net SD_DATA2: J302.69, J304.1 (DAT2)
- new net SD_DATA3: J302.61, J304.2 (DAT3/CD)
- new net SD_PWR: C303.1, J304.4 (VDD), U304.1 (VOUT)
- new net SD_PWR_ON: J302.75, R304.2, U304.4 (EN)
- new net TRD0+: J302.12, J303.2 (P2), U302.4 (D2+), U302.7 (NC)
- new net TRD0-: J302.10, J303.3 (P3), U302.5 (D2-), U302.6 (NC)
- new net TRD1+: J302.4, J303.4 (P4), U302.1 (D1+), U302.10 (NC)
- new net TRD1-: J302.6, J303.7 (P7), U302.2 (D1-), U302.9 (NC)
- new net TRD2+: J302.11, J303.5 (P5), U301.1 (D1+), U301.10 (NC)
- new net TRD2-: J302.9, J303.6 (P6), U301.2 (D1-), U301.9 (NC)
- new net TRD3+: J302.3, J303.8 (P8), U301.4 (D2+), U301.7 (NC)
- new net TRD3-: J302.5, J303.9 (P9), U301.5 (D2-), U301.6 (NC)
- new net USB+: J305.5
- new net USB-: J305.3
- new net USB_OTG_ID: R306.1
- no-connect marks 0 -> 117
Other:
- note added: "Ethernet: C54408"

Commit message: add hash and title
Other:
- note added: "Amateurfunkclub fuer Remote Stationen"
- note added: "CM4 (Raspberry Pi)"
- note added: "Remote Station"
Changed lines of the file:
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@@
+		)
+	)
+	(text "Remote Station"
+		(exclude_from_sim no)
+		(at 178.816 171.196 0)
+		(effects
+			(font
+				(size 5 5)
+			)
+			(justify left)
+		)
+	)
+	(text "Amateurfunkclub fuer Remote Stationen"
+		(exclude_from_sim no)
+		(at 186.436 189.992 0)
+		(effects
+			(font
+				(size 1.27 1.27)
+			)
+			(justify left)
+		)
+	)
+	(text "CM4 (Raspberry Pi)"
+		(exclude_from_sim no)
+		(at 179.07 178.054 0)
+		(effects
+			(font
+				(size 4 4)
+			)
+			(justify left)
 		)
 	)

Commit message: add hash
Other:
- note added: "<<HASH>>"
Changed lines of the file:
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@@
+		)
+	)
+	(text "<<HASH>>"
+		(exclude_from_sim no)
+		(at 267.97 193.548 0)
+		(effects
+			(font
+				(size 1.27 1.27)
+			)
+			(justify left)
 		)
 	)
