File: pcb/cm4/cm4-io.kicad_sch (KiCad schematic)
At the start: 11 parts, among them J301 Micro_SD_Card, J302 HR911130A, U301 RT9742GGJ5, U302 TPD4EUSB30, U303 TPD4EUSB30

Commit message: update cm4 board
Parts:
- renumbered C303 to C301, C301 to C302, C302 to C303, J302 to J301, J301 to J302, R302 to R301, R303 to R302, R301 to R303, U302 to U301, U303 to U302, U301 to U303
