File: pcb/bus/bus.kicad_pcb (KiCad board)
At the start: 4 copper layers, 117.4 x 100 mm, 36 parts, among them J201 Conn_02x10_Row_Letter_First, J301 Conn_02x10_Row_Letter_First, J401 Conn_02x10_Row_Letter_First, J501 Conn_02x10_Row_Letter_First, J601 Conn_02x10_Row_Letter_First, J701 Conn_02x10_Row_Letter_First, U101 USBLC6-2SC6, U102 FE1.1s, U103 USBLC6-2SC6, U104 USBLC6-2SC6, U105 USBLC6-2SC6, U106 USBLC6-2SC6, Y101 12MHz

Commit message: update bus pcb
Parts:
- added #SYM101: OSHW-Logo_7.5x8mm_SilkScreen, Symbol:OSHW-Logo_7.5x8mm_SilkScreen, F.Cu at (80.0, 106.2)
Routing:
- net /Device Connector 1/NS_USB-: track 6.79 -> 8.90 mm
- net /Device Connector 3/NS_USB+: track 7.48 -> 8.91 mm
- net /Device Connector 2/NS_USB+: track 7.55 -> 8.98 mm
- net /Device Connector 4/NS_USB+: track 7.41 -> 8.85 mm
- net /RPI Connector/NS_USB-: track 7.43 -> 8.84 mm
- net /USB2+: track 36.1 -> 37.3 mm
- net /USB1+: track 31.3 -> 32.4 mm
- net /Device Connector 1/NS_USB+: track 8.13 -> 8.94 mm
- net /USB4+: track 77.0 -> 77.8 mm
- net /USB3+: track 56.1 -> 56.9 mm
- net /MASTER_USB-: track 25.9 -> 26.6 mm
- net /Device Connector 3/NS_USB-: track 8.46 -> 9.00 mm
Other:
- board text added: "<<HASH>>"
- board text added: "Bus Board"
- board text added: "Copyright by {dblquote}Amateurfunkclub für Remote Stationen{dblquote} OE5XRX"
- board text added: "Device 1"
- board text added: "Device 2"
- board text added: "Device 3"
- board text added: "Device 4"
- board text added: "Power"
- board text added: "RPi"
