File: pcb/power/power_measurement.kicad_sch (KiCad schematic)
At the start: 3 parts, among them U301 INA226

Commit message: update ALL parts
Parts:
- C301: value 100nF -> 100n; LCSC C354365 -> C28233
- U301: LCSC (none) -> C49851
Changed lines of the file:
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@@
 			)
 		)
-		(property "Value" "100nF"
+		(property "Value" "100n"
 			(at 180.34 87.6299 0)
 			(effects
@@
 			)
 		)
-		(property "LCSC" "C354365"
-			(at 176.53 86.36 0)
-			(effects
-				(font
-					(size 1.27 1.27)
-				)
-				(hide yes)
+		(property "LCSC" "C28233"
+			(at 176.53 86.36 0)
+			(effects
+				(font
+					(size 1.27 1.27)
+				)
+				(hide yes)
+			)
+		)
+		(property "MOUSER" ""
+			(at 176.53 86.36 0)
+			(effects
+				(font
+					(size 1.27 1.27)
+				)
 			)
 		)
@@
 			)
 		)
+		(property "MOUSER" ""
+			(at 121.92 88.9 0)
+			(effects
+				(font
+					(size 1.27 1.27)
+				)
+			)
+		)
 		(pin "2"
 		)
@@
 			)
 		)
+		(property "LCSC" "C49851"
+			(at 143.51 90.17 0)
+			(effects
+				(font
+					(size 1.27 1.27)
+				)
+			)
+		)
+		(property "MOUSER" ""
+			(at 143.51 90.17 0)
+			(effects
+				(font
+					(size 1.27 1.27)
+				)
+			)
+		)

Commit message: update power pcb
Parts:
- R301: value 100m -> 10m; LCSC C2903476 -> (none)
Changed lines of the file:
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@@
 			)
 		)
-		(property "Value" "100m"
+		(property "Value" "10m"
 			(at 124.46 90.1699 0)
 			(effects
@@
 			)
 		)
-		(property "LCSC" "C2903476"
+		(property "LCSC" ""
 			(at 121.92 88.9 0)
 			(effects
