File: pcb/power/power_measurement.kicad_sch (KiCad schematic)
At the start: 3 parts, among them U301 INA226

Commit message: update fields and mouser components
Parts:
- R301: MOUSER (none) -> 652-CRF2512FZR010ELF
Changed lines of the file:
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@@
 			)
 		)
-		(property "MOUSER" ""
+		(property "MOUSER" "652-CRF2512FZR010ELF"
 			(at 121.92 88.9 0)
 			(effects
@@
 					(size 1.27 1.27)
 				)
+				(hide yes)
 			)
 		)
