File: pcb/power/5V.kicad_sch (KiCad schematic)
At the start: 13 parts, among them U203 LMR51430 500kHz

Commit message: update fields and mouser components
Parts:
- L201: LCSC C167231 -> (none); MOUSER (none) -> 710-74439346068
- R202: MOUSER (none) -> 603-RC0805JR-07100KL
- R203: MOUSER (none) -> 652-CR0805FX-1372ELF
- U203: MOUSER (none) -> 595-LMR51430XDDCR
Changed lines of the file:
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@@
 			)
 		)
-		(property "LCSC" "C167231"
+		(property "LCSC" ""
 			(at 168.91 78.74 0)
 			(effects
@@
 			)
 		)
-		(property "MOUSER" ""
+		(property "MOUSER" "710-74439346068"
 			(at 168.91 78.74 0)
 			(effects
@@
 					(size 1.27 1.27)
 				)
+				(hide yes)
 			)
 		)
@@
 			)
 		)
-		(property "MOUSER" ""
+		(property "MOUSER" "603-RC0805JR-07100KL"
 			(at 173.99 92.71 0)
 			(effects
@@
 			)
 		)
+		(property "MOUSER" "595-LMR51430XDDCR"
+			(at 133.35 81.28 0)
+			(effects
+				(font
+					(size 1.27 1.27)
+				)
+				(hide yes)
+			)
+		)
 		(pin "1"
 		)
@@
 			)
 		)
-		(property "MOUSER" ""
+		(property "MOUSER" "652-CR0805FX-1372ELF"
 			(at 173.99 102.87 0)
 			(effects
