File: pcb/power/power.kicad_sch (KiCad schematic)
At the start: 14 parts, among them J101 XT60PW-M, J102 Conn_02x10_Row_Letter_First

Commit message: update fields and mouser components
Parts:
- F101, F102, F103: LCSC C19727304 -> (none); MOUSER (none) -> 576-01530007Z
- J101: Height 8.4 -> (none); Manufacturer_Name Amass -> (none); Manufacturer_Part_Number XT60PW-M -> (none)
Changed lines of the file:
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@@
-			)
-		)
-		(property "Sim.Pins" "1=K 2=A"
-			(at 86.36 147.32 0)
-			(effects
-				(font
-					(size 1.27 1.27)
-				)
-				(hide yes)
 			)
 		)
@@
 			)
 		)
-		(property "Sim.Pins" "1=K 2=A"
-			(at 71.12 147.32 0)
-			(effects
-				(font
-					(size 1.27 1.27)
-				)
-				(hide yes)
-			)
-		)
 		(property "MOUSER" ""
 			(at 71.12 147.32 0)
@@
 			)
 		)
-		(property "Height" "8.4"
-			(at 49.53 427.94 0)
-			(effects
-				(font
-					(size 1.27 1.27)
-				)
-				(justify left top)
-				(hide yes)
-			)
-		)
-		(property "TME Electronic Components Part Number" ""
-			(at 49.53 527.94 0)
-			(effects
-				(font
-					(size 1.27 1.27)
-				)
-				(justify left top)
-				(hide yes)
-			)
-		)
-		(property "TME Electronic Components Price/Stock" ""
-			(at 49.53 627.94 0)
-			(effects
-				(font
-					(size 1.27 1.27)
-				)
-				(justify left top)
-				(hide yes)
-			)
-		)
-		(property "Manufacturer_Name" "Amass"
-			(at 49.53 727.94 0)
-			(effects
-				(font
-					(size 1.27 1.27)
-				)
-				(justify left top)
-				(hide yes)
-			)
-		)
-		(property "Manufacturer_Part_Number" "XT60PW-M"
-			(at 49.53 827.94 0)
-			(effects
-				(font
-					(size 1.27 1.27)
-				)
-				(justify left top)
-				(hide yes)
-			)
-		)
 		(property "LCSC" ""
 			(at 30.48 33.02 0)
@@
 			)
 		)
-		(property "LCSC" "C19727304"
+		(property "LCSC" ""
 			(at 156.21 34.29 0)
 			(effects
@@
 			)
 		)
-		(property "MOUSER" ""
+		(property "MOUSER" "576-01530007Z"
 			(at 156.21 34.29 0)
 			(effects
@@
 					(size 1.27 1.27)
 				)
+				(hide yes)
 			)
 		)
@@
 			)
 		)
-		(property "LCSC" "C19727304"
+		(property "LCSC" ""
 			(at 80.01 39.37 0)
 			(effects
@@
 			)
 		)
-		(property "MOUSER" ""
+		(property "MOUSER" "576-01530007Z"
 			(at 80.01 39.37 0)
 			(effects
@@
 					(size 1.27 1.27)
 				)
+				(hide yes)
 			)
 		)
@@
 			)
 		)
-		(property "LCSC" "C19727304"
+		(property "LCSC" ""
 			(at 156.21 76.2 0)
 			(effects
@@
 			)
 		)
-		(property "MOUSER" ""
+		(property "MOUSER" "576-01530007Z"
 			(at 156.21 76.2 0)
 			(effects
@@
 					(size 1.27 1.27)
 				)
-			)
-		)
+				(hide yes)
+			)
+		)
