File: pcb/fm/AF_OUT-ADC-filter.kicad_sch (KiCad schematic)
At the start: 5 parts

Commit message: update fm module
Parts:
- R403: LCSC (none) -> C17520
Changed lines of the file:
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@@
 			)
 		)
-		(property "LCSC" ""
+		(property "LCSC" "C17520"
 			(at 163.83 90.17 0)
 			(effects
