File: pcb/fm/DAC-MIC_IN-filter.kicad_sch (KiCad schematic)
At the start: 7 parts

Commit message: update fm module
Parts:
- C302, C303: value 5.9nF -> 5.6nF/X7R/100V; MOUSER (none) -> 791-0805B562K201CT
- R301: MOUSER (none) -> 603-RT0805DRE0756KL
- R302, R303, R304: MOUSER (none) -> 603-RT0805DRE0710KL
Changed lines of the file:
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@@
 			)
 		)
-		(property "MOUSER" ""
+		(property "MOUSER" "603-RT0805DRE0710KL"
 			(at 177.8 81.28 0)
 			(effects
@@
 			)
 		)
-		(property "MOUSER" ""
+		(property "MOUSER" "603-RT0805DRE0710KL"
 			(at 160.02 81.28 0)
 			(effects
@@
 			)
 		)
-		(property "MOUSER" ""
+		(property "MOUSER" "603-RT0805DRE0756KL"
 			(at 124.46 73.66 90)
 			(effects
@@
 			)
 		)
-		(property "Value" "5.9nF"
+		(property "Value" "5.6nF/X7R/100V"
 			(at 193.04 90.1699 0)
 			(effects
@@
 			)
 		)
+		(property "MOUSER" "791-0805B562K201CT"
+			(at 189.23 88.9 0)
+			(effects
+				(font
+					(size 1.27 1.27)
+				)
+				(hide yes)
+			)
+		)
 		(pin "2"
 		)
@@
 			)
 		)
-		(property "MOUSER" ""
+		(property "MOUSER" "603-RT0805DRE0710KL"
 			(at 124.46 88.9 0)
 			(effects
@@
 			)
 		)
-		(property "Value" "5.9nF"
+		(property "Value" "5.6nF/X7R/100V"
 			(at 172.72 90.1699 0)
 			(effects
@@
 			(at 168.91 88.9 0)
 			(effects
+				(font
+					(size 1.27 1.27)
+				)
+				(hide yes)
+			)
+		)
+		(property "MOUSER" "791-0805B562K201CT"
+			(at 168.91 88.9 0)
+			(effects
