File: pcb/fm/connector_cpu.kicad_sch (KiCad schematic)
At the start: 15 parts, among them J101 Conn_02x10_Row_Letter_First, J201 Conn_ARM_JTAG_SWD_10, U201 STM32F302CBTx, U202 TLV73333PQDBVRQ1, U203 CAT24C32, Y201 8MHz / 20pF

Commit message: update fm pcb
Connections:
- no-connect marks 19 -> 27

Commit message: add title block to fm module
Other:
- company: (none) -> Amateurfunkclub für Remote Stationen
- title: (none) -> STM32
Changed lines of the file:
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@@
 	(generator_version "9.0")
 	(paper "A4")
+	(title_block
+		(title "STM32")
+		(rev "<<HASH>>")
+		(company "Amateurfunkclub für Remote Stationen")
+	)
 	(junction
 		(at 189.23 127)

Commit message: update fm module
Parts:
- added C202, C204, C206, C208, C210, C214: 100nF, Capacitor_SMD:C_0805_2012Metric, symbol Device:C
- added C207, C209: 4.7u/10V/X5R, Capacitor_SMD:C_0805_2012Metric, symbol Device:C
- C201: LCSC (none) -> C28233
- C203: renamed from C202; value 22pF -> 30pF; MOUSER (none) -> 791-0805N300J500CT
- C205: renamed from C203; value 22pF -> 30pF; MOUSER (none) -> 791-0805N300J500CT
- C211: renamed from C204; MOUSER (none) -> 791-0805B105K250CT
- C212: renamed from C205; MOUSER (none) -> 791-0805B105K250CT
- R201: LCSC (none) -> C17520
- R202: MOUSER (none) -> 603-RT0805DRD073K9L
- U201: MOUSER (none) -> 511-STM32F302CBT7
- U202: renamed from U203; MOUSER (none) -> 698-CAT24C32WI-GT3
- Y201: MOUSER (none) -> 73-XT49M800-20
- renumbered C101 to C213, J101 to J202, U202 to U203
Connections:
- net +3V3: now also C202.2, C204.2, C206.2, C207.2, C208.2, C209.2, C214.2
- net +5V: now also C210.2
- net GND: now also C202.1, C204.1, C206.1, C207.1, C208.1, C209.1, C210.1, C214.1
Other:
- moved on the sheet: C201, C203, C205, C211, C212, C213, J201, J202, JP201, R201, R202, U201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

Commit message: update fm module
Parts:
- added C215: 100nF, Capacitor_SMD:C_0805_2012Metric, symbol Device:C
- added U204: USBLC6-2SC6, Package_TO_SOT_SMD:SOT-23-6, symbol Power_Protection:USBLC6-2SC6
Connections:
- net +3V3: now also C215.1, U204.5 (VBUS)
- net GND: now also C215.2, U204.2 (GND)
- net USB_D_N renamed NS_USB-
- net NS_USB-: now also U204.3 (I/O2); no longer J202.b6 (Pin_b6)
- net USB_D_P renamed NS_USB+
- net NS_USB+: now also U204.1 (I/O1); no longer J202.a6 (Pin_a6)
- new net USB+: J202.a6 (Pin_a6), U204.6 (I/O1)
- new net USB-: J202.b6 (Pin_b6), U204.4 (I/O2)
