File: pcb/fm/fm.kicad_pcb (KiCad board)
At the start: 4 copper layers, 100 x 100 mm, 46 parts, among them J101 Conn_02x10_Row_Letter_First, J102 Conn_Coaxial, J201 Conn_ARM_JTAG_SWD_10, Q101 2N7002, Q102 2N7002, Q103 2N7002, U101 SA818V, U102 XC6227C401PR-G, U201 STM32F302CBTx, U202 TLV73333PQDBVRQ1, U203 CAT24C32, Y201 8MHz / 20pF

Commit message: update fm pcb
Parts:
- moved C101 7.18 mm to (184.5, 87.8)
- moved U203 6.11 mm to (171.6, 69.7)
- moved C205 5.13 mm to (177.7, 80.3), turned to 90 degrees
- moved R202 4.81 mm to (177.8, 72.3), turned to 0 degrees
- moved C109 4.62 mm to (176.4, 108.7)
- moved Q101 4.62 mm to (179.7, 108.4)
- moved C204 4.60 mm to (184.7, 81.0), turned to 90 degrees
- moved C102 4.28 mm to (117.3, 101.7), turned to 180 degrees
- moved JP201 3.65 mm to (177.8, 69.6)
- moved C103 2.97 mm to (113.5, 101.7), turned to 0 degrees
- moved C111 2.55 mm to (172.6, 103.7)
- moved Q103 2.43 mm to (175.8, 103.7)
- moved C110 2.16 mm to (166.6, 107.0)
- moved Q102 2.03 mm to (169.8, 107.1)
- moved U102 1.62 mm to (115.4, 105.6)
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Routing:
- net +3V3: track 0.00 -> 177.2 mm, vias 0 -> 6
- net /Connector and CPU/SWCLK: track 0.00 -> 133.6 mm, vias 0 -> 2
- net /Connector and CPU/SWDIO: track 0.00 -> 117.8 mm, vias 0 -> 2
- net +5V: track 10.2 -> 113.4 mm, vias 0 -> 2
- net GND: track 0.00 -> 75.1 mm, vias 0 -> 24
- net /Connector and CPU/nRESET: track 0.00 -> 73.5 mm, vias 0 -> 3
- net /H_L_Power: track 0.00 -> 70.6 mm
- net /nPOWER_DOWN: track 0.00 -> 65.0 mm
- net /nPTT: track 0.00 -> 49.2 mm
- net /RADIO_RX: track 0.00 -> 47.3 mm, vias 0 -> 2
- net /MIC_IN: track 0.00 -> 42.9 mm, vias 0 -> 2
- net /RADIO_TX: track 0.00 -> 39.2 mm, vias 0 -> 2
- net /nSQUELCH: track 0.00 -> 35.7 mm, vias 0 -> 2
- net /AF_OUT: track 0.00 -> 29.8 mm
- net Net-(U201-PF0): track 0.00 -> 19.8 mm
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- added copper zone on In1.Cu, net GND
- added copper zone on In2.Cu, net GND

Commit message: update fm module
Parts:
- removed C107, C108, C109, C110, C111: 10nF/NP0, Capacitor_SMD:C_0805_2012Metric
- removed J102: Conn_Coaxial, Connector_Coaxial:SMA_Amphenol_132289_EdgeMount
- removed Q101, Q102, Q103: 2N7002, Package_TO_SOT_SMD:SOT-23
- removed R103, R109, R110: 220, Resistor_SMD:R_0805_2012Metric
- removed R104, R108: 10k, Resistor_SMD:R_0805_2012Metric
- removed R105: 2k2, Resistor_SMD:R_0805_2012Metric
- removed R106, R107: 5k1, Resistor_SMD:R_0805_2012Metric
- added C206: 100nF, Capacitor_SMD:C_0805_2012Metric, F.Cu at (164.6, 80.8)
- added C207: 4.7u/10V/X5R, Capacitor_SMD:C_0805_2012Metric, F.Cu at (164.6, 83.0)
- added C208: 100nF, Capacitor_SMD:C_0805_2012Metric, F.Cu at (160.5, 90.5)
- added C209: 4.7u/10V/X5R, Capacitor_SMD:C_0805_2012Metric, F.Cu at (160.5, 92.7)
- added C210: 100nF, Capacitor_SMD:C_0805_2012Metric, F.Cu at (184.7, 81.0)
- added C211: 1uF, Capacitor_SMD:C_0805_2012Metric, F.Cu at (186.8, 81.0)
- added C212: 1uF, Capacitor_SMD:C_0805_2012Metric, F.Cu at (177.5, 80.3)
- added C213: 100u / 25V, Capacitor_Tantalum_SMD:CP_EIA-7343-43_Kemet-X, F.Cu at (184.5, 87.7)
- added C214: 100nF, Capacitor_SMD:C_0805_2012Metric, F.Cu at (177.0, 77.5)
- added C301: 4.7u/10V/X5R, Capacitor_SMD:C_0805_2012Metric, F.Cu at (169.9, 100.9)
- added C302: 5.9nF, Capacitor_SMD:C_0805_2012Metric, F.Cu at (163.8, 100.9)
- added C303: 5.9nF, Capacitor_SMD:C_0805_2012Metric, F.Cu at (165.9, 104.5)
- added C401: 4.7u/10V/X5R, Capacitor_SMD:C_0805_2012Metric, F.Cu at (157.0, 99.1)
- added C402: 10nF/NP0, Capacitor_SMD:C_0805_2012Metric, F.Cu at (160.5, 94.8)
- added C501: 10nF/NP0, Capacitor_SMD:C_0805_2012Metric, F.Cu at (127.8, 106.8)
- added C601: 10nF/NP0, Capacitor_SMD:C_0805_2012Metric, F.Cu at (145.4, 104.1)
- added C701: 10nF/NP0, Capacitor_SMD:C_0805_2012Metric, F.Cu at (135.1, 104.5)
- added J202: Conn_02x10_Row_Letter_First, PRJ:PCN10C-20S-2.54DS, F.Cu at (191.6, 74.8)
- added Q501: 2N7002, Package_TO_SOT_SMD:SOT-23, F.Cu at (130.9, 107.8)
- added Q601: 2N7002, Package_TO_SOT_SMD:SOT-23, F.Cu at (148.6, 105.2)
- added Q701: 2N7002, Package_TO_SOT_SMD:SOT-23, F.Cu at (138.3, 105.6)
- added R301: 56k, Resistor_SMD:R_0805_2012Metric, F.Cu at (169.9, 97.4)
- added R302: 10k, Resistor_SMD:R_0805_2012Metric, F.Cu at (167.9, 97.4)
- added R303: 10k, Resistor_SMD:R_0805_2012Metric, F.Cu at (167.9, 100.9)
- added R304: 10k, Resistor_SMD:R_0805_2012Metric, F.Cu at (165.9, 100.9)
- added R401: 5k1, Resistor_SMD:R_0805_2012Metric, F.Cu at (157.0, 97.0)
- added R402: 5k1, Resistor_SMD:R_0805_2012Metric, F.Cu at (160.5, 99.1)
- added R403: 2k2, Resistor_SMD:R_0805_2012Metric, F.Cu at (160.5, 97.0)
- added R501: 10k, Resistor_SMD:R_0805_2012Metric, F.Cu at (134.8, 108.7)
- added R601: 10k, Resistor_SMD:R_0805_2012Metric, F.Cu at (152.5, 106.1)
- added R701: 10k, Resistor_SMD:R_0805_2012Metric, F.Cu at (142.2, 106.6)
- C101: value 100u / 25V -> 100nF; footprint Capacitor_Tantalum_SMD:CP_EIA-7343-43_Kemet-X -> Capacitor_SMD:C_0805_2012Metric
- C102: value 1uF -> 10uF
- C103: value 2.2uF -> 10nF/NP0
- C104: value 100nF -> 1uF
- C105: value 4.7u/10V/X5R -> 2.2uF
- C106: value 4.7u/10V/X5R -> 100nF
- C202: value 22pF -> 100nF
- C203: value 22pF -> 30pF
- C204: value 1uF -> 100nF
- C205: value 1uF -> 30pF
- J101: value Conn_02x10_Row_Letter_First -> Conn_Coaxial; footprint PRJ:PCN10C-20S-2.54DS -> Connector_Coaxial:SMA_Amphenol_132289_EdgeMount
- R101, R102: value 10k -> 220
- U202: value TLV73333PQDBVRQ1 -> CAT24C32; footprint Package_TO_SOT_SMD:SOT-23-5 -> Package_SO:SOIC-8_3.9x4.9mm_P1.27mm
- U203: value CAT24C32 -> TLV73333PQDBVRQ1; footprint Package_SO:SOIC-8_3.9x4.9mm_P1.27mm -> Package_TO_SOT_SMD:SOT-23-5
- moved J101 91.2 mm to (100.5, 77.5), turned to 180 degrees
- moved C101 75.7 mm to (109.1, 94.1)
- moved C103 58.8 mm to (172.3, 103.2), turned to 90 degrees
- moved C104 50.0 mm to (116.5, 107.5), turned to -90 degrees
- moved C105 48.6 mm to (116.5, 111.6)
- moved C106 44.9 mm to (114.3, 111.6), turned to -90 degrees
- moved C202 29.5 mm to (176.9, 93.3), turned to 180 degrees
- moved C205 28.1 mm to (152.9, 93.7), turned to -90 degrees
- moved R101 19.3 mm to (173.2, 78.9)
- moved R102 18.9 mm to (171.2, 78.9)
- moved C203 17.5 mm to (152.9, 76.3), turned to 90 degrees
- moved U202 14.4 mm to (171.6, 69.5), turned to -90 degrees
- moved U203 14.3 mm to (181.1, 80.3), turned to 180 degrees
- moved C204 8.04 mm to (176.9, 83.1), turned to 180 degrees
- moved U102 6.33 mm to (120.4, 109.5), turned to 180 degrees
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Connections:
- C101 pad 1: +5V -> GND
- C101 pad 2: GND -> +4V
- C102 pad 1: +5V -> GND
- C102 pad 2: GND -> +4V
- C103 pad 1: +4V -> GND
- C103 pad 2: GND -> /nSQUELCH
- C104 pad 1: GND -> +5V
- C104 pad 2: Net-(C104-Pad2) -> GND
- C105 pad 1: /MIC_IN -> +4V
- C105 pad 2: Net-(C104-Pad2) -> GND
- C106 pad 1: Net-(C106-Pad1) -> GND
- C106 pad 2: /AF_OUT -> +4V
- C202 pad 1: Net-(U201-PF0) -> GND
- C202 pad 2: GND -> +3V3
- C203 pad 1: Net-(U201-PF1) -> Net-(U201-PF0)
- C204 pad 1: +5V -> GND
- C204 pad 2: GND -> +3V3
- C205 pad 1: +3V3 -> Net-(U201-PF1)
- R101 pad 1: /GPIO3 -> /RADIO_RX
- R101 pad 2: Net-(Q101-G) -> /Connector and CPU/USART_TX
- R102 pad 1: /GPIO1 -> /RADIO_TX
- R102 pad 2: Net-(Q102-G) -> /Connector and CPU/USART_RX
- U202 pad 1: +5V -> GND
- U202 pad 3: +5V -> GND
- U202 pad 4: unconnected-(U202-NC-Pad4) -> GND
- U202 pad 5: +3V3 -> /Connector and CPU/I2C_SDA_MEM
- U203 pad 1: GND -> +5V
- U203 pad 3: GND -> +5V
- U203 pad 4: GND -> unconnected-(U203-NC-Pad4)
- U203 pad 5: /Connector and CPU/I2C_SDA_MEM -> +3V3
Routing:
- net /H_L_Power: track 70.6 -> 18.3 mm
- net /GPIO3: track 8.71 -> 59.7 mm
- net /nPOWER_DOWN: track 65.0 -> 20.8 mm
- net /GPIO2: track 7.05 -> 50.3 mm
- net GND: track 75.1 -> 116.9 mm, vias 24 -> 30
- net /GPIO1: track 5.40 -> 37.5 mm
- net +3V3: track 177.2 -> 146.4 mm, vias 6 -> 7
- net /nPTT: track 49.2 -> 26.1 mm
- net +4V: track 9.35 -> 26.2 mm
- net +5V: track 113.4 -> 124.4 mm, vias 2 -> 3
- net Net-(Q101-G): track 10.1 -> 0.00 mm
- net Net-(Q102-G): track 8.57 -> 0.00 mm
- net Net-(C401-Pad1): track 0.00 -> 7.76 mm
- net Net-(C104-Pad2): track 6.06 -> 0.00 mm
- net /AF_OUT: track 29.8 -> 24.1 mm
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
Commit message: update fm module
Parts:
- removed C105: 2.2uF, Capacitor_SMD:C_0805_2012Metric
- removed C106: 100nF, Capacitor_SMD:C_0805_2012Metric
- removed U102: XC6227C401PR-G, Package_TO_SOT_SMD:SOT-89-5
- added C215: 100nF, Capacitor_SMD:C_0805_2012Metric, F.Cu at (183.5, 88.1)
- added C802: 10u, Capacitor_SMD:C_1206_3216Metric, F.Cu at (134.6, 118.1)
- added C803: 10u, Capacitor_SMD:C_1206_3216Metric, F.Cu at (131.9, 118.1)
- added C804: 100n, Capacitor_SMD:C_0805_2012Metric, F.Cu at (129.4, 118.6)
- added C805: 100n, Capacitor_SMD:C_0805_2012Metric, F.Cu at (121.6, 119.2)
- added C806: 22u, Capacitor_SMD:C_1206_3216Metric, F.Cu at (117.9, 119.6)
- added C807: 22u, Capacitor_SMD:C_1206_3216Metric, F.Cu at (117.9, 116.9)
- added C808: 100n, Capacitor_SMD:C_0805_2012Metric, F.Cu at (118.4, 114.4)
- added L801: 6.8u, PRJ:WE-XHMI_6060, F.Cu at (119.4, 125.6)
- added R801: 49R9, Resistor_SMD:R_0805_2012Metric, F.Cu at (130.4, 113.0)
- added R802: 100k, Resistor_SMD:R_0805_2012Metric, F.Cu at (127.3, 114.0)
- added R803: 13k7, Resistor_SMD:R_0805_2012Metric, F.Cu at (125.0, 114.0)
- added U204: USBLC6-2SC6, Package_TO_SOT_SMD:SOT-23-6, F.Cu at (180.3, 87.1)
- added U801: LMR51430 500kHz, Package_TO_SOT_SMD:SOT-23-6, F.Cu at (126.0, 118.4)
- C104: value 1uF -> 100u / 25V; footprint Capacitor_SMD:C_0805_2012Metric -> Capacitor_Tantalum_SMD:CP_EIA-7343-43_Kemet-X
- C302, C303: value 5.9nF -> 5.6nF/X7R/100V
- moved C104 23.8 mm to (138.4, 116.8), turned to 90 degrees
- moved C213 14.3 mm to (183.4, 73.5), turned to 90 degrees
- moved C101 6.75 mm to (110.5, 100.7), turned to 0 degrees
- moved C102 2.81 mm to (110.5, 102.9)
Connections:
- net +4V renamed +5V_HF
- C104 pad 1: +5V -> +12V
- J202 pad a6: /Connector and CPU/USB_D_P -> /Connector and CPU/USB+
- J202 pad b6: /Connector and CPU/USB_D_N -> /Connector and CPU/USB-
- U201 pad 32: /Connector and CPU/USB_D_N -> /Connector and CPU/NS_USB-
- U201 pad 33: /Connector and CPU/USB_D_P -> /Connector and CPU/NS_USB+
Routing:
- net +5V: track 124.4 -> 25.0 mm, vias 3 -> 2
- net +3V3: track 146.4 -> 182.2 mm, vias 7 -> 9
- net /Connector and CPU/USB_D_N: track 18.6 -> 0.00 mm
- net /Connector and CPU/USB_D_P: track 17.6 -> 0.00 mm
- net +12V: track 10.2 -> 21.6 mm, vias 0 -> 2
- net /Connector and CPU/USB+: track 0.00 -> 10.8 mm
- net /Connector and CPU/USB-: track 0.00 -> 10.7 mm
- net /Connector and CPU/SWDIO: track 117.8 -> 127.3 mm, vias 2 -> 1
- net Net-(U801-CB): track 0.00 -> 6.20 mm, vias 0 -> 2
- net /Connector and CPU/SWCLK: track 133.6 -> 139.7 mm, vias 2 -> 1
- net Net-(U801-FB): track 0.00 -> 4.81 mm
- net /Connector and CPU/NS_USB-: track 0.00 -> 4.79 mm
- net /Connector and CPU/NS_USB+: track 0.00 -> 4.78 mm
- net +5V_HF: track 26.2 -> 30.2 mm, vias 0 -> 2
- net GND: track 116.9 -> 112.9 mm, vias 30 -> 45
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- added copper zone on F.Cu, net +12V
- added copper zone on F.Cu, net +5V
- added copper zone on F.Cu, net +5V_HF
- added copper zone on F.Cu, net /5V/TPS_SW
- added copper zone on F.Cu, net GND

Commit message: update fm pcb
Parts:
- moved C601 16.0 mm to (129.8, 100.7), turned to 180 degrees
- moved C701 11.7 mm to (124.1, 100.7), turned to 180 degrees
- moved C501 10.9 mm to (118.7, 100.7), turned to 180 degrees
- moved #SYM101 7.68 mm to (115.2, 55.8)
Routing:
- net GND: track 112.9 -> 86.6 mm, vias 45 -> 114
- net /Connector and CPU/nRESET: track 73.7 -> 76.0 mm
- net /H_L_Power: track 18.3 -> 20.0 mm
- net /Connector and CPU/SWCLK: track 139.7 -> 138.5 mm
- net /Connector and CPU/SWDIO: track 127.3 -> 126.3 mm
- net /nPOWER_DOWN: track 20.8 -> 21.6 mm
- net /RADIO_RX: track 47.3 -> 46.4 mm
- net /MIC_IN: track 48.5 -> 49.1 mm
