File: pcb/fm/fm.kicad_sch (KiCad schematic)
At the start: 30 parts, among them J102 Conn_Coaxial, Q101 2N7002, Q102 2N7002, Q103 2N7002, U101 SA818V, U102 XC6227C401PR-G

Commit message: add title block to fm module
Other:
- company: (none) -> Amateurfunkclub für Remote Stationen
- title: (none) -> FM Module
Changed lines of the file:
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@@
 	(generator_version "9.0")
 	(paper "A4")
+	(title_block
+		(title "FM Module")
+		(rev "<<HASH>>")
+		(company "Amateurfunkclub für Remote Stationen")
+	)
 	(junction
 		(at 137.16 38.1)

Commit message: update fm module
Parts:
- removed C104: 100nF, Capacitor_SMD:C_0805_2012Metric, symbol Device:C
- removed C105: 4.7u/10V/X5R, Capacitor_SMD:C_0805_2012Metric, symbol Device:C
- removed C107, C109, C110, C111: 10nF/NP0, Capacitor_SMD:C_0805_2012Metric, symbol Device:C
- removed Q101, Q102, Q103: 2N7002, Package_TO_SOT_SMD:SOT-23, symbol Transistor_FET:2N7002
- removed R101, R102, R104, R108: 10k, Resistor_SMD:R_0805_2012Metric, symbol Device:R
- removed R103: 220, Resistor_SMD:R_0805_2012Metric, symbol Device:R
- removed R105: 2k2, Resistor_SMD:R_0805_2012Metric, symbol Device:R
- removed R106, R107: 5k1, Resistor_SMD:R_0805_2012Metric, symbol Device:R
- added C101: 100nF, Capacitor_SMD:C_0805_2012Metric, symbol Device:C
- added C102: 10uF, Capacitor_SMD:C_0805_2012Metric, symbol Device:C
- C103: renamed from C108; MOUSER (none) -> 81-GRM2165C2A103JA1D
- C104: renamed from C102; MOUSER (none) -> 791-0805B105K250CT
- C105: renamed from C103; MOUSER (none) -> 187-CL21B225KOFNNNG
- C106: value 4.7u/10V/X5R -> 100nF; LCSC (none) -> C28233
- D101: MOUSER (none) -> 78-BAT43W-G3-08
- FL101: MOUSER (none) -> 139-LFCN-180 / 139-LFCN-490
- J101: renamed from J102; MOUSER (none) -> 530-142-0701-801
- R101: renamed from R110; MOUSER (none) -> 667-ERA-6AEB221V
- R102: renamed from R109; MOUSER (none) -> 667-ERA-6AEB221V
- U101: LCSC (none) -> C3001504
- U102: MOUSER (none) -> 865-XC6227C401PR-G
Connections:
- net +4V: now also C106.2, C101.2, C102.2
- net AF_OUT: no longer C106.2
- net GND: now also C106.1, C101.1, C102.1
Other:
- added sheet AF_OUT to ADC filter (AF_OUT-ADC-filter.kicad_sch)
- added sheet DAC to MIC_IN filter (DAC-MIC_IN-filter.kicad_sch)
- added sheet Pin Driver SA818 (pin_driver.kicad_sch)
- added sheet Pin Driver SA819 (pin_driver.kicad_sch)
- added sheet Pin Driver SA820 (pin_driver.kicad_sch)
- moved on the sheet: C104, C105, U102

Commit message: update fm module
Parts:
- removed C104: 1uF, Capacitor_SMD:C_0805_2012Metric, symbol Device:C
- removed C105: 2.2uF, Capacitor_SMD:C_0805_2012Metric, symbol Device:C
- removed C106: 100nF, Capacitor_SMD:C_0805_2012Metric, symbol Device:C
- removed U102: XC6227C401PR-G, Package_TO_SOT_SMD:SOT-89-5, symbol Regulator_Linear:XC6220B331MR
Connections:
- net +4V renamed +5V_HF
Other:
- added sheet 5V (5V.kicad_sch)

Commit message: multiple fixes
Parts:
- U101: SnapEDA_Link https://www.snapeda.com/parts/DRA818V/DORJI/view-part/?ref=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 -> (none)
Changed lines of the file:
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@@
-			)
-		)
-		(property "SnapEDA_Link" "https://www.snapeda.com/parts/DRA818V/DORJI/view-part/?ref=snap"
-			(at 60.96 103.124 0)
-			(effects
-				(font
-					(size 1.27 1.27)
-				)
-				(justify bottom)
-				(hide yes)
 			)
 		)

Commit message: fix multiple inventree parts
Parts:
- FL101: MOUSER 139-LFCN-180 / 139-LFCN-490 -> 139-LFCN-180,139-LFCN-490
Changed lines of the file:
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@@
 			)
 		)
-		(property "MOUSER" "139-LFCN-180 / 139-LFCN-490"
+		(property "MOUSER" "139-LFCN-180,139-LFCN-490"
 			(at 58.42 152.4 0)
 			(effects
